Commit message: Removed reusnake_visualize reference

File: src/snake_monster/urdf/rotary_module.xacro (robot description, xacro)
@@ -9,5 +9,5 @@
 	<origin xyz="0 0 -0.035" rpy="-1.57075 0 0" />
         <geometry>
-          <mesh filename="package://reusnake_visualize/meshes/rotary_input.stl"/>
+          <mesh filename="package://snake_monster/meshes/rotary_input.stl"/>
         </geometry>
         <xacro:red_material/>
@@ -51,5 +51,5 @@
         <origin xyz="0 0 0" rpy="-1.57075 0 0" />
         <geometry>
-          <mesh filename="package://reusnake_visualize/meshes/rotary_output.stl"/>
+          <mesh filename="package://snake_monster/meshes/rotary_output.stl"/>
 	  <!-- <cylinder radius=".0025" length=".1" /> -->
         </geometry>

Commit message: wrap around open-loop works

File: src/snake_monster/urdf/rotary_module.xacro (robot description, xacro)
@@ -33,5 +33,5 @@
       <axis xyz="0 1 0"/>
       <dynamics damping=".1" friction="0.2"/>
-      <limit effort="7.0" lower="-1.57" upper="1.57" velocity="2.208932"/>
+      <limit effort="20.0" lower="-1.57" upper="1.57" velocity="2.208932"/>
     </joint>
     <transmission name="${name}_trans">

Commit message: changed actuator values to correct maximum effort

File: src/snake_monster/urdf/rotary_module.xacro (robot description, xacro)
@@ -33,5 +33,5 @@
       <axis xyz="0 1 0"/>
       <dynamics damping=".1" friction="0.2"/>
-      <limit effort="20.0" lower="-1.57" upper="1.57" velocity="2.208932"/>
+      <limit effort="7.0" lower="-1.57" upper="1.57" velocity="2.208932"/>
     </joint>
     <transmission name="${name}_trans">

Commit message: new gait_3.py for compliant, compliant working

File: src/snake_monster/urdf/rotary_module.xacro (robot description, xacro)
@@ -33,5 +33,5 @@
       <axis xyz="0 1 0"/>
       <dynamics damping=".1" friction="0.2"/>
-      <limit effort="7.0" lower="-1.57" upper="1.57" velocity="2.208932"/>
+      <limit effort="5.0" lower="-1.57" upper="1.57" velocity="2.208932"/>
     </joint>
     <transmission name="${name}_trans">

Commit message: added fake effort generator to test compliance. compliance is working with fake effort generator

File: src/snake_monster/urdf/rotary_module.xacro (robot description, xacro)
@@ -33,5 +33,5 @@
       <axis xyz="0 1 0"/>
       <dynamics damping=".1" friction="0.2"/>
-      <limit effort="5.0" lower="-1.57" upper="1.57" velocity="2.208932"/>
+      <limit effort="4.0" lower="-1.57" upper="1.57" velocity="2.208932"/>
     </joint>
     <transmission name="${name}_trans">

Commit message: gaits_3.py is working with full compliance

File: src/snake_monster/urdf/rotary_module.xacro (robot description, xacro)
@@ -33,5 +33,5 @@
       <axis xyz="0 1 0"/>
       <dynamics damping=".1" friction="0.2"/>
-      <limit effort="4.0" lower="-1.57" upper="1.57" velocity="2.208932"/>
+      <limit effort="5.0" lower="-1.57" upper="1.57" velocity="2.208932"/>
     </joint>
     <transmission name="${name}_trans">

Commit message: finished all_the_same data collection

File: src/snake_monster/urdf/rotary_module.xacro (robot description, xacro)
@@ -33,5 +33,5 @@
       <axis xyz="0 1 0"/>
       <dynamics damping=".1" friction="0.2"/>
-      <limit effort="10.0" lower="-1.57" upper="1.57" velocity="2.208932"/>
+      <limit effort="7.0" lower="-1.57" upper="1.57" velocity="2.208932"/>
     </joint>
     <transmission name="${name}_trans">
