Commit message: Changed urdf to match reusnake conventions, modified gait script, added camera

File: src/snake_control/urdf/snake.xacro (robot description, xacro)
@@ -6,4 +6,5 @@
   <xacro:include filename="./module_common.xacro"/>
   <xacro:include filename="./rotary_module.xacro"/>
+  <xacro:include filename="./realsense-RS200.macro.xacro"/>
   <!-- ************************* ROBOT DEFINITION ************************* -->
   <xacro:property name="S_00" value="SA001__MoJo" />
@@ -23,20 +24,26 @@
   <xacro:property name="S_14" value="SA015__MoJo" />
   <xacro:property name="S_15" value="SA016__MoJo" />
+  <!-- Import all Gazebo-customization elements -->
+  <xacro:include filename="./snake.gazebo" />
   <link name="kdl_dummy_root" />
   <joint name="kdl_dummy_root_to_base" type="fixed">
     <parent link="kdl_dummy_root"/>
     <child link="base"/>
-    <origin xyz="0 0 0" rpy="0 ${-PI/2.0} 0"/>
+    <origin xyz="0 0 0" rpy="0 -${PI/2} 0"/>
   </joint>
   <!-- base body -->
   <link name="base" />
+  <joint name = "base_to_camera" type="fixed">
+    <parent link="base" />
+    <child link="camera_link" />
+    <origin xyz="0 0 0" rpy="0 ${-PI/2} 0"/>
+  </joint>
+  <link name="camera_link"/>
   <!-- leg outputs on the base -->
   <joint name="head__OUTPUT_INTERFACE" type="fixed">
     <parent link="base"/>
     <child link="${S_00}__INPUT_INTERFACE"/>
-    <!-- <origin xyz="${width/2} ${leg_y_offset} ${height/2}" rpy="-${PI/2} 0 -${PI/2}"/> -->
+    <origin xyz="0 0 0" rpy="0 0 -${PI/2}"/> -->
   </joint>
-  <!-- Import all Gazebo-customization elements -->
-  <xacro:include filename="./snake.gazebo" />
   <xacro:rotary_module joint="${S_00}" child="${S_01}"/>
   <xacro:rotary_module joint="${S_01}" child="${S_02}"/>

File: src/snake_monster/urdf/rotary_module.xacro (robot description, xacro)
@@ -3,16 +3,16 @@
   <xacro:property name="mass_2" value=".103" />
   <xacro:property name="cyl_r" value=".026" />
-  <xacro:property name="cyl_h" value=".033" />
+  <xacro:property name="cyl_h" value="-0.033" />
   <xacro:macro name="rotary_module_in" params="name">
     <link name="${name}">
       <visual>
-	<origin xyz="0 0 0.035" rpy="1.57075 0 0" />
+	<origin xyz="0 0 -0.035" rpy="-1.57075 0 0" />
         <geometry>
-          <mesh filename="package://snake_monster/meshes/rotary_input.stl"/>
+          <mesh filename="package://reusnake_visualize/meshes/rotary_input.stl"/>
         </geometry>
         <xacro:red_material/>
       </visual>
     <collision>
-      <origin xyz="0 0 ${0.0366/2.0}" rpy="0 0 0" />
+      <origin xyz="0 0 -${0.0366/2.0}" rpy="0 0 0" />
       <geometry>
 	<cylinder radius="${cyl_r}" length="${cyl_h}" />
@@ -20,5 +20,5 @@
     </collision>
     <inertial>
-      <origin xyz="0 0 0.0366" rpy="0 0 0" />
+      <origin xyz="0 0 -0.0366" rpy="0 0 0" />
       <mass value="${mass_2}"/>
       <inertia ixx="${mass_2/12.0*(3*cyl_r**2+cyl_h**2)+mass_2*(cyl_h/2.0)**2}" iyy="${mass_2/12.0*(3*cyl_r**2+cyl_h**2)+mass_2*(cyl_h/2.0)**2}" izz="${mass_2/2.0*cyl_r**2}" ixy="0" ixz="0" iyz="0" />
@@ -30,5 +30,5 @@
       <parent link="${parent}"/>
       <child link="${child}"/>
-      <origin xyz="0 0 0.0366" rpy="0 0 0"/>
+      <origin xyz="0 0 -0.0366" rpy="0 0 0"/>
       <axis xyz="0 1 0"/>
       <dynamics damping=".1" friction="0.2"/>
@@ -49,7 +49,7 @@
     <link name="${name}">
       <visual>
-        <origin xyz="0 0 0" rpy="1.57075 0 0" />
+        <origin xyz="0 0 0" rpy="-1.57075 0 0" />
         <geometry>
-          <mesh filename="package://snake_monster/meshes/rotary_output.stl"/>
+          <mesh filename="package://reusnake_visualize/meshes/rotary_output.stl"/>
 	  <!-- <cylinder radius=".0025" length=".1" /> -->
         </geometry>
@@ -57,5 +57,5 @@
       </visual>
     <collision>
-      <origin xyz="0 0 ${0.0366/2.0}" rpy="0 0 0" />
+      <origin xyz="0 0 -${0.0366/2.0}" rpy="0 0 0" />
       <geometry>
 	<cylinder radius="${cyl_r}" length="${cyl_h}" />
@@ -73,5 +73,5 @@
       <parent link="${parent}"/>
       <child link="${child}"/>
-      <origin xyz="0 0 0.0273" rpy="0 0 -1.57075"/>
+      <origin xyz="0 0 -0.0273" rpy="0 0 -1.57075"/>
     </joint>
   </xacro:macro>

Commit message: Modified camera frame to match head frame during VO

File: src/snake_control/urdf/snake.xacro (robot description, xacro)
@@ -34,8 +34,15 @@
   <!-- base body -->
   <link name="base" />
+  <!--
   <joint name = "base_to_camera" type="fixed">
     <parent link="base" />
     <child link="camera_link" />
     <origin xyz="0 0 0" rpy="0 ${-PI/2} 0"/>
+  </joint>
+  -->
+  <joint name = "base_to_camera" type="fixed">
+    <parent link="base" />
+    <child link="camera_link" />
+    <origin xyz="0 0 0" rpy="0 ${-PI/2} ${PI/2}"/>
   </joint>
   <link name="camera_link"/>
