Commit message: working

File: src/snake_control/urdf/rotary_module_vluu.xacro (robot description, xacro)
@@ -11,5 +11,5 @@
           <mesh filename="package://snake_monster/meshes/rotary_input.stl"/>
         </geometry>
-        <xacro:red_material/>
+        <xacro:black_material/>
       </visual>
     <collision>
@@ -33,5 +33,5 @@
       <axis xyz="0 1 0"/>
       <dynamics damping=".1" friction="0.2"/>
-      <limit effort="10.0" lower="-1.57" upper="1.57" velocity="2.208932"/>
+      <limit effort="5.0" lower="-1.57" upper="1.57" velocity="2.208932"/>
     </joint>
     <transmission name="${name}_trans">
@@ -54,5 +54,5 @@
 	  <!-- <cylinder radius=".0025" length=".1" /> -->
         </geometry>
-        <xacro:red_material/>
+        <xacro:black_material/>
       </visual>
     <collision>
